File: Production Files/RedBot-Panel-v11.brd (EAGLE design)
At the start: 94 x 99.6 mm, 129 parts, among them U1 ATMEGA328P, U10 MIC5219 5V, U11 MIC5219 3.3V, U12 7408SE, U2 TB6612FNG, U3 MIC5219 5V, U4 MIC5219 3.3V, U5 FT232RLSSOP, U6 7408SE, U7 ATMEGA328P, U8 FT232RLSSOP, U9 TB6612FNG, Y1 16MHz, Y2 16MHz

Commit message: Panelized v11 board
Parts:
- turned D11 to 90 degrees
- turned D3 to 90 degrees
- turned D5 to 90 degrees
- turned D9 to 90 degrees
Connections:
- removed net N$13 (its old number): D11.A, R18.1
- removed net N$14 (its old number): D9.A, R17.1
- new net N$21: D11.C, R18.1
- new net N$22: D9.C, R17.1
- net GND: no longer D3.C, D5.C
- net GND1: no longer D11.C, D9.C
- net N$3: now also D5.C; no longer D5.A
- net N$4: now also D3.C; no longer D3.A
- net V_USB: now also D3.A, D5.A
- net V_USB1: now also D11.A, D9.A
Routing:
- net GND1: track 84.7 -> 82.2 mm, vias 44 -> 43
- net GND: track 84.7 -> 82.2 mm, vias 44 -> 43
- net V_USB1: track 43.5 -> 45.7 mm
- net V_USB: track 43.5 -> 45.7 mm
- net N$22: track 0.00 -> 1.14 mm
- net N$21: track 0.00 -> 1.14 mm
- net N$14 (its old number): track 1.14 -> 0.00 mm
- net N$13 (its old number): track 1.14 -> 0.00 mm
Other:
- board text added: "v11"
- board text removed: "v10"
