File: Production Files/RedBot-Panel-v12.brd (EAGLE design)
At the start: 94 x 99.6 mm, 129 parts, among them U1 ATMEGA328P, U10 MIC5219 5V, U11 MIC5219 3.3V, U12 7408SE, U2 TB6612FNG, U3 MIC5219 5V, U4 MIC5219 3.3V, U5 FT232RLSSOP, U6 7408SE, U7 ATMEGA328P, U8 FT232RLSSOP, U9 TB6612FNG, Y1 16MHz, Y2 16MHz

Commit message: Created v12 panel
Parts:
- C1, C10, C11, C12, C13, C14, C2, C3, C4, C5, C6, C7: device SparkFun-Capacitors:0402-CAP -> SparkFun-Capacitors:0603-CAP
- R1, R10, R11, R12, R13, R14, R15, R16, R17, R18, R19, R2, R20, R21, R22, R23, R24, R25, R26, R3, R4, R5, R6, R7, R8, R9: device SparkFun-Resistors:0402-RES -> SparkFun-Resistors:0603-RES
- moved R1 0.51 mm to (54.0, 20.2)
- moved R14 0.51 mm to (54.0, 70.2)
- moved C14 0.38 mm to (54.0, 69.0)
- moved D11 0.38 mm to (76.6, 66.5)
- moved D3 0.38 mm to (76.6, 15.2)
- moved D5 0.38 mm to (76.6, 16.5)
- moved D9 0.38 mm to (76.6, 65.3)
- moved R19 0.38 mm to (62.2, 77.1)
- moved C7 0.38 mm to (54.0, 18.9)
- moved R7 0.38 mm to (62.2, 27.1)
- moved C1 0.25 mm to (40.3, 79.6)
- moved C10 0.25 mm to (53.7, 77.2)
- moved C2 0.25 mm to (40.3, 29.6)
- moved C3 0.25 mm to (53.7, 27.2)
- moved D12 0.25 mm to (56.9, 95.8)
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Routing:
- net FT232_RXI1: track 43.4 -> 42.5 mm
- net FT232_RXI: track 43.4 -> 42.5 mm
- net 5V: track 62.1 -> 61.4 mm
- net 5V1: track 62.1 -> 61.4 mm
- net SCK: track 23.4 -> 22.8 mm
- net SCK1: track 23.4 -> 22.8 mm
- net V_BATT1: track 80.8 -> 81.3 mm
- net V_BATT: track 80.8 -> 81.3 mm
Other:
- board text added: "v12"
- board text removed: "v11"
